File: PCB/hackpad.kicad_sch (KiCad schematic)
At the start: 35 parts, among them SW11 SW_Push, SW12 SW_Push, SW13 SW_Push, SW14 SW_Push, SW15 SW_Push, SW16 SW_Push, SW17 SW_Push, SW18 SW_Push, SW19 SW_Push, SW4 RotaryEncoder_Switch, U1 MOUDLE-SEEEDUINO-XIAO, U2 ER_OLEDM0.91_1x-I2C

Commit message: PCB Update
Parts:
- removed D13: 1N4148, Diode_THT:D_DO-35_SOD27_P7.62mm_Horizontal, symbol Diode:1N4148
Connections:
- net at SW17.1, SW18.1, SW19.1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: no longer SW4.S2
- net at D23.1 (K), U1.4 (PA11_A3_D3): now also D20.1 (K), D28.1 (K); no longer D25.1 (K), D27.1 (K)
- net at D22.1 (K), U1.9 (PA7_A8_D8_SCK): now also D26.1 (K), D27.1 (K); no longer D20.1 (K), D21.1 (K)
- net at D24.1 (K), U1.8 (PB09_A7_D7_RX): now also D21.1 (K), D25.1 (K); no longer D26.1 (K), D28.1 (K)
- no-connect marks 4 -> 9
Other:
- moved on the sheet: D20, D21, D22, D23, D25, D27, SW12, SW13, SW17, SW18, SW19

Commit message: Add files via upload
Connections:
- net at D21.1 (K), D25.1 (K), U1.8 (PB09_A7_D7_RX): now also D26.1 (K); no longer D24.1 (K)
- net at D20.1 (K), D23.1 (K): now also D24.1 (K), U1.9 (PA7_A8_D8_SCK); no longer D28.1 (K), U1.4 (PA11_A3_D3)
- net at D22.1 (K), D27.1 (K): now also D28.1 (K), U1.4 (PA11_A3_D3); no longer D26.1 (K), U1.9 (PA7_A8_D8_SCK)

Commit message: Add files via upload
Connections:
- net at D2.2 (DIN), U1.7 (PB08_A6_D6_TX): no longer D3.2 (DIN), D4.2 (DIN)
- net row2: now reaches D9.4 (DOUT)
- net row2: now also D4.2 (DIN)
- net row1: now reaches D8.4 (DOUT)
- net row1: now also D3.2 (DIN)
- no-connect marks 9 -> 7
Other:
- moved on the sheet: D10, D4, D5, D6, D7, D8, D9
